File: ESC-logic.kicad_pcb (KiCad board)
At the start: 4 copper layers, 50 x 50 mm, 68 parts, among them J1 CAN, J10 Conn_01x02, J2 USB_C, J3 HALL, J4 COMM, J5 SERVO, J6 SWD, J7 SENSE, J8 CURRENT, J9 GATE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

Commit message: Changed jst connectors
Parts:
- J1: footprint Connector_JST:JST_PH_B4B-PH-K_1x04_P2.00mm_Vertical -> Connector_JST:JST_PH_S4B-PH-K_1x04_P2.00mm_Horizontal
- J3: footprint Connector_JST:JST_PH_B6B-PH-K_1x06_P2.00mm_Vertical -> Connector_JST:JST_PH_S6B-PH-K_1x06_P2.00mm_Horizontal
- J4: footprint Connector_JST:JST_PH_B7B-PH-K_1x07_P2.00mm_Vertical -> Connector_JST:JST_PH_S7B-PH-K_1x07_P2.00mm_Horizontal
- J5: footprint Connector_JST:JST_PH_B3B-PH-K_1x03_P2.00mm_Vertical -> Connector_JST:JST_PH_S3B-PH-K_1x03_P2.00mm_Horizontal
- J6: footprint Connector_JST:JST_PH_B5B-PH-K_1x05_P2.00mm_Vertical -> Connector_JST:JST_PH_S5B-PH-K_1x05_P2.00mm_Horizontal
- moved R6 3.45 mm to (131.9, 92.2)
- moved C45 3.08 mm to (117.5, 109.0)
- moved R24 3.08 mm to (119.5, 109.0)
- moved R25 3.08 mm to (121.5, 109.0)
- moved R27 3.08 mm to (123.5, 109.0)
- moved R28 3.08 mm to (125.5, 109.0)
- moved J1 2.21 mm to (103.2, 103.2)
- moved J5 2.20 mm to (103.2, 94.2)
- moved C4 2.17 mm to (111.0, 83.2)
- moved J6 2.15 mm to (103.2, 81.3)
- moved C7 2.07 mm to (111.0, 85.2)
- moved J3 2.00 mm to (114.9, 113.0)
- moved J4 2.00 mm to (129.8, 113.0)
- moved Q1 1.96 mm to (132.0, 94.8), turned to 180 degrees
- moved C39 1.95 mm to (146.5, 112.2), turned to -90 degrees
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Connections:
- J7 pad 2: +5V -> GND
- J7 pad 8: GND -> +12V
- J9 pad 1: /MCU/H1 -> /MCU/H3
- J9 pad 2: GND -> /MCU/H2
- J9 pad 3: /MCU/H2 -> GND
- J9 pad 4: /MCU/H3 -> /MCU/H1
- J9 pad 5: /MCU/L1 -> /MCU/L3
- J9 pad 7: /MCU/L3 -> +5V
- J9 pad 8: +12V -> /MCU/L1
- U2 pad 34: /MCU/L3 -> /MCU/L1
- U2 pad 36: /MCU/L1 -> /MCU/L3
- U2 pad 41: /MCU/H3 -> /MCU/H1
- U2 pad 43: /MCU/H1 -> /MCU/H3
Routing:
- net +5V: track 93.9 -> 109.1 mm, vias 2 -> 3
- net +12V: track 44.9 -> 53.9 mm, vias 0 -> 1
- net GND: track 4.91 -> 11.3 mm, vias 11 -> 13
- net Net-(Q1-Pad3): track 13.9 -> 19.5 mm
- net /MCU/AN_IN: track 26.7 -> 21.2 mm
- net /MCU/L1: track 13.3 -> 17.6 mm
- net /MCU/H3: track 16.9 -> 12.6 mm
- net /MCU/H1: track 12.6 -> 16.9 mm
- net /Hall/TEMP_IN: track 30.8 -> 34.6 mm
- net +3V3: track 249.4 -> 252.3 mm
- net /MCU/NRST: track 21.3 -> 18.6 mm
- net /MCU/H2: track 13.4 -> 16.0 mm
- net /MCU/MISO_ADC_EXT2: track 39.1 -> 41.3 mm
- net /MCU/TX_SCL_MOSI: track 39.9 -> 37.9 mm
- net /MCU/RX_SDA_NSS: track 46.1 -> 48.1 mm
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
Commit message: what changed?
Parts:
- added N1: Housing, Symbol:KiCad-Logo2_5mm_SilkScreen, F.Cu at (117.8, 85.5)
- C10, C11, C3, C4, C5, C7, C8, C9: value 2.2u -> 2u2
- moved C45 7.75 mm to (125.2, 108.8), turned to -90 degrees
- moved R25 4.26 mm to (117.2, 108.8)
- moved R27 4.26 mm to (119.2, 108.8)
- moved R28 4.26 mm to (121.2, 108.8)
- moved R24 3.76 mm to (123.2, 108.8)
- turned U9 to 0 degrees
Connections:
- J1 pad 1: +5V -> GND
- J1 pad 2: /CAN/CAN_H -> /CAN/CAN_L
- J1 pad 3: /CAN/CAN_L -> /CAN/CAN_H
- J1 pad 4: GND -> +5V
- J3 pad 2: /Hall/TEMP_IN -> /Hall/HALL3_IN
- J3 pad 3: /Hall/HALL3_IN -> /Hall/HALL2_IN
- J3 pad 4: /Hall/HALL2_IN -> /Hall/HALL1_IN
- J3 pad 5: /Hall/HALL1_IN -> /Hall/TEMP_IN
- J5 pad 2: Net-(J5-Pad2) -> +5V
- J5 pad 3: +3V3 -> Net-(J5-Pin_3)
- J6 pad 1: +3V3 -> /MCU/NRST
- J6 pad 2: /MCU/SWCLK -> /MCU/SWDIO
- J6 pad 4: /MCU/SWDIO -> /MCU/SWCLK
- J6 pad 5: /MCU/NRST -> +3V3
- R40 pad 1: Net-(J5-Pad2) -> Net-(J5-Pin_3)
- U9 pad 1: +3V3 -> GND
- U9 pad 2: GND -> +5V
- U9 pad 3: +5V -> +3V3
Routing:
- net +3V3: track 252.3 -> 237.9 mm, vias 6 -> 7
- net +5V: track 109.1 -> 121.3 mm
- net /MCU/NRST: track 18.6 -> 27.8 mm
- net /Hall/TEMP_IN: track 34.6 -> 28.5 mm
- net Net-(J5-Pin_3): track 0.00 -> 5.72 mm
- net /CAN/CAN_L: track 10.3 -> 14.6 mm
- net Net-(J5-Pad2): track 2.83 -> 0.00 mm
- net GND: track 11.3 -> 14.1 mm, vias 13 -> 16
- net /Hall/HALL1_IN: track 32.6 -> 30.0 mm
- net /Hall/HALL2_IN: track 31.7 -> 29.4 mm
- net /MCU/SWCLK: track 11.3 -> 9.63 mm
- net /Hall/HALL3_IN: track 31.7 -> 30.0 mm
- net /CAN/CAN_H: track 14.9 -> 13.7 mm
- net /MCU/SWDIO: track 14.2 -> 15.4 mm, vias 1 -> 0
- net /MCU/CURRENT_C: track 23.2 -> 23.8 mm
Other:
- board text added: "ESC-logic v0.1 9/12/22"
- board text added: "JLCJLCJLCJLC"
