File: ESC-logic.kicad_sch (KiCad schematic)
At the start: 20 parts, among them J1 CAN, J10 Conn_01x02, J2 USB_C, J3 HALL, J4 COMM, J5 SERVO, J6 SWD, J7 SENSE, J8 CURRENT, J9 GATE

Commit message: Changed jst connectors
Parts:
- J1: footprint Connector_JST:JST_PH_B4B-PH-K_1x04_P2.00mm_Vertical -> Connector_JST:JST_PH_S4B-PH-K_1x04_P2.00mm_Horizontal
- J3: footprint Connector_JST:JST_PH_B6B-PH-K_1x06_P2.00mm_Vertical -> Connector_JST:JST_PH_S6B-PH-K_1x06_P2.00mm_Horizontal
- J4: footprint Connector_JST:JST_PH_B7B-PH-K_1x07_P2.00mm_Vertical -> Connector_JST:JST_PH_S7B-PH-K_1x07_P2.00mm_Horizontal
- J5: footprint Connector_JST:JST_PH_B3B-PH-K_1x03_P2.00mm_Vertical -> Connector_JST:JST_PH_S3B-PH-K_1x03_P2.00mm_Horizontal
- J6: footprint Connector_JST:JST_PH_B5B-PH-K_1x05_P2.00mm_Vertical -> Connector_JST:JST_PH_S5B-PH-K_1x05_P2.00mm_Horizontal
Connections:
- net +12V: now also J7.8 (Pin_8); no longer J9.8 (Pin_8)
- net +5V: now also J9.7 (Pin_7); no longer J7.2 (Pin_2)
- net GND: now also J7.2 (Pin_2), J9.3 (Pin_3); no longer J7.8 (Pin_8), J9.2 (Pin_2)
- net MCU/H1: now also J9.4 (Pin_4); no longer J9.1 (Pin_1)
- net MCU/H2: now also J9.2 (Pin_2); no longer J9.3 (Pin_3)
- net MCU/H3: now also J9.1 (Pin_1); no longer J9.4 (Pin_4)
- net MCU/L1: now also J9.8 (Pin_8); no longer J9.5 (Pin_5)
- net MCU/L3: now also J9.5 (Pin_5); no longer J9.7 (Pin_7)

Commit message: what changed?
Parts:
- added N1: Housing, Symbol:KiCad-Logo2_5mm_SilkScreen, symbol Mechanical:Housing
- C49: LCSC (none) -> C49678
- J2: LCSC (none) -> C709357
- R40: LCSC (none) -> C105577
- R7, R8: LCSC (none) -> C84375
Connections:
- net +3V3: now also J6.5 (Pin_5); no longer J5.3 (Pin_3), J6.1 (Pin_1)
- net +5V: now also J1.4 (Pin_4), J5.2 (Pin_2); no longer J1.1 (Pin_1)
- net CAN/CAN_H: now also J1.3 (Pin_3); no longer J1.2 (Pin_2)
- net CAN/CAN_L: now also J1.2 (Pin_2); no longer J1.3 (Pin_3)
- net GND: now also J1.1 (Pin_1); no longer J1.4 (Pin_4)
- net Hall/HALL1_IN: now also J3.4 (Pin_4); no longer J3.5 (Pin_5)
- net Hall/HALL2_IN: now also J3.3 (Pin_3); no longer J3.4 (Pin_4)
- net Hall/HALL3_IN: now also J3.2 (Pin_2); no longer J3.3 (Pin_3)
- net Hall/TEMP_IN: now also J3.5 (Pin_5); no longer J3.2 (Pin_2)
- net MCU/NRST: now also J6.1 (Pin_1); no longer J6.5 (Pin_5)
- net MCU/SWCLK: now also J6.4 (Pin_4); no longer J6.2 (Pin_2)
- net MCU/SWDIO: now also J6.2 (Pin_2); no longer J6.4 (Pin_4)
- net at R40.1: now also J5.3 (Pin_3); no longer J5.2 (Pin_2)
Other:
- note added: "Low pass filter: 15.92 KHz"
- moved on the sheet: J5
