File: Power.kicad_sch (KiCad schematic)
At the start: 25 parts, among them U7 SY8502, U8 ZTP7193Y, U9 SE8533

Commit message: Changed jst connectors
Parts:
- removed R19, R3: R, symbol Device:R
Changed lines of the file:
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@@
   (junction (at 78.74 82.55) (diameter 0) (color 0 0 0 0)
   )
-  (junction (at 181.61 133.35) (diameter 0) (color 0 0 0 0)
-  )
   (junction (at 114.3 151.13) (diameter 0) (color 0 0 0 0)
   )
@@
     (stroke (width 0) (type default) (color 0 0 0 0))
   )
-  (wire (pts (xy 181.61 130.81) (xy 181.61 133.35))
-    (stroke (width 0) (type default) (color 0 0 0 0))
-  )
   (wire (pts (xy 52.07 125.73) (xy 67.31 125.73))
     (stroke (width 0) (type default) (color 0 0 0 0))
@@
     (stroke (width 0) (type default) (color 0 0 0 0))
   )
-  (wire (pts (xy 181.61 133.35) (xy 181.61 137.16))
-    (stroke (width 0) (type default) (color 0 0 0 0))
-  )
   (wire (pts (xy 66.04 64.77) (xy 69.85 64.77))
     (stroke (width 0) (type default) (color 0 0 0 0))
@@
     (stroke (width 0) (type default) (color 0 0 0 0))
   )
-  (wire (pts (xy 200.66 133.35) (xy 181.61 133.35))
-    (stroke (width 0) (type default) (color 0 0 0 0))
-  )
-  (wire (pts (xy 181.61 121.92) (xy 181.61 123.19))
-    (stroke (width 0) (type default) (color 0 0 0 0))
-  )
   (wire (pts (xy 114.3 88.9) (xy 114.3 91.44))
     (stroke (width 0) (type default) (color 0 0 0 0))
@@
     (stroke (width 0) (type default) (color 0 0 0 0))
   )
-  (wire (pts (xy 200.66 124.46) (xy 200.66 133.35))
-    (stroke (width 0) (type default) (color 0 0 0 0))
-  )
   (wire (pts (xy 97.79 60.96) (xy 97.79 64.77))
     (stroke (width 0) (type default) (color 0 0 0 0))
@@
   )
   (wire (pts (xy 67.31 148.59) (xy 67.31 149.86))
-    (stroke (width 0) (type default) (color 0 0 0 0))
-  )
-  (wire (pts (xy 181.61 144.78) (xy 181.61 147.32))
     (stroke (width 0) (type default) (color 0 0 0 0))
   )
@@
   (label "ZTP_EN" (at 55.88 137.16 0)
     (effects (font (size 0.8 0.8)) (justify left bottom))
-  )
-  (global_label "1V65" (shape input) (at 200.66 124.46 90) (fields_autoplaced)
-    (effects (font (size 1.27 1.27)) (justify left))
-    (property "Intersheet References" "${INTERSHEET_REFS}" (id 0) (at 200.5806 117.3298 90)
-      (effects (font (size 1.27 1.27)) (justify left) hide)
-    )
   )
   (global_label "V_SUPPLY" (shape input) (at 30.48 60.96 180) (fields_autoplaced)
@@
     (pin "1")
   )
-  (symbol (lib_id "Device:R") (at 181.61 127 0) (unit 1)
-    (in_bom yes) (on_board yes) (fields_autoplaced)
-    (property "Reference" "R3" (id 0) (at 184.15 125.7299 0)
-      (effects (font (size 1.27 1.27)) (justify left))
-    )
-    (property "Value" "R" (id 1) (at 184.15 128.2699 0)
-      (effects (font (size 1.27 1.27)) (justify left))
-    )
-    (property "Footprint" "" (id 2) (at 179.832 127 90)
-      (effects (font (size 1.27 1.27)) hide)
-    )
-    (property "Datasheet" "~" (id 3) (at 181.61 127 0)
-      (effects (font (size 1.27 1.27)) hide)
-    )
-    (pin "1")
-    (pin "2")
-  )
-  (symbol (lib_id "Device:R") (at 181.61 140.97 0) (unit 1)
-    (in_bom yes) (on_board yes) (fields_autoplaced)
-    (property "Reference" "R19" (id 0) (at 184.15 139.6999 0)
-      (effects (font (size 1.27 1.27)) (justify left))
-    )
-    (property "Value" "R" (id 1) (at 184.15 142.2399 0)
-      (effects (font (size 1.27 1.27)) (justify left))
-    )
-    (property "Footprint" "" (id 2) (at 179.832 140.97 90)
-      (effects (font (size 1.27 1.27)) hide)
-    )
-    (property "Datasheet" "~" (id 3) (at 181.61 140.97 0)
-      (effects (font (size 1.27 1.27)) hide)
-    )
-    (pin "1")
-    (pin "2")
-  )
   (symbol (lib_id "Device:R") (at 114.3 85.09 0) (unit 1)
     (in_bom yes) (on_board yes)
@@
     (pin "1")
   )
-  (symbol (lib_id "power:+3V3") (at 181.61 121.92 0) (unit 1)
-    (in_bom yes) (on_board yes) (fields_autoplaced)
-    (property "Reference" "#PWR0115" (id 0) (at 181.61 125.73 0)
-      (effects (font (size 1.27 1.27)) hide)
-    )
-    (property "Value" "+3V3" (id 1) (at 184.15 120.6499 0)
-      (effects (font (size 1.27 1.27)) (justify left))
-    )
-    (property "Footprint" "" (id 2) (at 181.61 121.92 0)
-      (effects (font (size 1.27 1.27)) hide)
-    )
-    (property "Datasheet" "" (id 3) (at 181.61 121.92 0)
-      (effects (font (size 1.27 1.27)) hide)
-    )
-    (pin "1")
-  )
   (symbol (lib_id "power:+5V") (at 190.5 68.58 0) (unit 1)
     (in_bom yes) (on_board yes) (fields_autoplaced)
@@
     (pin "2")
   )
-  (symbol (lib_id "power:GND") (at 181.61 147.32 0) (unit 1)
-    (in_bom yes) (on_board yes) (fields_autoplaced)
-    (property "Reference" "#PWR0113" (id 0) (at 181.61 153.67 0)
-      (effects (font (size 1.27 1.27)) hide)
-    )
-    (property "Value" "GND" (id 1) (at 181.61 152.4 0))
-    (property "Footprint" "" (id 2) (at 181.61 147.32 0)
-      (effects (font (size 1.27 1.27)) hide)
-    )
-    (property "Datasheet" "" (id 3) (at 181.61 147.32 0)
-      (effects (font (size 1.27 1.27)) hide)
-    )
-    (pin "1")
-  )
   (symbol (lib_id "Device:C_Small") (at 91.44 78.74 0) (mirror y) (unit 1)

Commit message: what changed?
Parts:
- C28, C32, C35: LCSC C386093 -> C45783
- C30, C33: LCSC (none) -> C319195
- C39: LCSC C962154 -> C15850
- R18: LCSC (none) -> C180850
- R22: LCSC (none) -> C2930184
Connections:
- net +3V3: now also U9.3 (VOUT); no longer U9.1 (VOUT)
- net +5V: now also U9.2 (VIN); no longer U9.3 (VIN)
- net GND: now also U9.1 (GND); no longer U9.2 (GND)
Other:
- note added: "R on enable pin not necessary C 220n on input not usefull, replace with second 2,2uF"
- note added: "Switching frequency 395kHz"
